Commit message: Wrist roll added in XACRO file

File: urdf/bhimbot_five_dof_arm.xacro (robot description, xacro)
@@ -28,4 +28,6 @@
 <property name="elbow_pitch_width" value="0.04" />
 <property name="elbow_pitch_height" value="0.04" />
+<property name="wrist_roll_width" value="0.06" />
+<property name="wrist_roll_len" value="0.02" />
 <!-- //////////////////////////////////////////////////////////////////////////////////////////////////////////////////////  -->
   <link name="bottom_link">
@@ -55,7 +57,7 @@
     <parent link="base_link" />
     <child link="shoulder_pan_link" />
-    <origin xyz="0 0 0.04" rpy="0 ${M_PI/2} ${M_PI*0}" />
+    <origin xyz="0 0 0.04" rpy="-${M_PI/2} ${M_PI/2} ${M_PI*0}" />
     <axis xyz="-1 0 0" />
-    <limit effort="300" velocity="1" lower="-2.61799387799" upper="1.98394848567" />
+    <limit effort="300" velocity="1" lower="-1.57" upper="1.57" />
   </joint>
   <link name="shoulder_pan_link">
@@ -72,6 +74,6 @@
     <child link="shoulder_pitch_link" />
     <origin xyz="-0.041 0.0021 0.0" rpy="-${M_PI/2} 0 ${M_PI/2}" />
-    <axis xyz="1 0 0" />
-    <limit effort="300" velocity="1" lower="-1.19962513147" upper="1.89994105047" />
+    <axis xyz="0 1 0" />
+    <limit effort="300" velocity="1" lower="-1.57" upper="1.57" />
   </joint>
   <link name="shoulder_pitch_link">
@@ -87,7 +89,7 @@
     <parent link="shoulder_pitch_link" />
     <child link="elbow_pitch_link" />
-    <origin xyz="0 0 0.11" rpy="${M_PI/2} 0 0" />
+    <origin xyz="0 0 0.11" rpy="0 0 ${M_PI/2}" />
     <axis xyz="1 0 0" />
-    <limit effort="300" velocity="1" lower="-1.5953400194" upper="1.93281579274" />
+    <limit effort="300" velocity="1" lower="-1.57" upper="1.57" />
   </joint>
   <link name="elbow_pitch_link">
@@ -97,4 +99,21 @@
         <box size="${elbow_pitch_len} ${elbow_pitch_width} ${elbow_pitch_height}" />
       </geometry>
+      <material name="White" />
+    </visual>
+  </link>
+  <joint name="wrist_roll_joint" type="revolute">
+    <parent link="elbow_pitch_link" />
+    <child link="wrist_roll_link"/>
+    <origin xyz="0 0 0.22" rpy="-${M_PI/2} ${M_PI/2} 0" />
+    <axis xyz="-1 0 0" />
+    <limit effort="300" velocity="1" lower="-1.57" upper="1.57" />
+  </joint>
+  <link name="wrist_roll_link">
+    <visual>
+      <origin xyz="0 0 0" rpy="0 ${M_PI/2} 0"/>
+      <geometry>
+        <cylinder radius="${wrist_roll_width}" length="${wrist_roll_len}" />
+      </geometry>
+      <material name="Grey" />
     </visual>
   </link>

Commit message: Modified XACRO file: added wrist pitch link, gripper, etc

File: urdf/bhimbot_five_dof_arm.xacro (robot description, xacro)
@@ -28,10 +28,16 @@
 <property name="elbow_pitch_width" value="0.04" />
 <property name="elbow_pitch_height" value="0.04" />
+<property name="wrist_pitch_len" value="0.10" />
+<property name="wrist_pitch_width" value="0.04" />
+<property name="wrist_pitch_height" value="0.04" />
 <property name="wrist_roll_width" value="0.06" />
 <property name="wrist_roll_len" value="0.02" />
+<property name="gripper_finger_len" value="0.08" />
+<property name="gripper_finger_width" value="0.01" />
+<property name="gripper_finger_height" value="0.01" />
 <!-- //////////////////////////////////////////////////////////////////////////////////////////////////////////////////////  -->
   <link name="bottom_link">
     <visual>
-      <origin xyz="0 0 -0.04" rpy="0 0 0" />
+      <origin xyz="0 0 -0.01" rpy="0 0 0" />
       <geometry>
         <box size="1 1 0.02" />
@@ -47,5 +53,5 @@
   <link name="base_link">
     <visual>
-      <origin xyz="0 0 0" rpy="0 0 0" />
+      <origin xyz="0 0 0.03" rpy="0 0 0" />
       <geometry>
         <cylinder radius="${base_width}" length="${base_len}" />
@@ -57,5 +63,5 @@
     <parent link="base_link" />
     <child link="shoulder_pan_link" />
-    <origin xyz="0 0 0.04" rpy="-${M_PI/2} ${M_PI/2} ${M_PI*0}" />
+    <origin xyz="0 0 0.07" rpy="-${M_PI/2} ${M_PI/2} ${M_PI*0}" />
     <axis xyz="-1 0 0" />
     <limit effort="300" velocity="1" lower="-1.57" upper="1.57" />
@@ -73,5 +79,5 @@
     <parent link="shoulder_pan_link" />
     <child link="shoulder_pitch_link" />
-    <origin xyz="-0.041 0.0021 0.0" rpy="-${M_PI/2} 0 ${M_PI/2}" />
+    <origin xyz="0 0 0" rpy="-${M_PI/2} 0 ${M_PI/2}" />
     <axis xyz="0 1 0" />
     <limit effort="300" velocity="1" lower="-1.57" upper="1.57" />
@@ -79,5 +85,5 @@
   <link name="shoulder_pitch_link">
     <visual>
-      <origin xyz="-0.002 0 0.04" rpy="0 ${M_PI/2} 0" />
+      <origin xyz="0 0 0.07" rpy="0 ${M_PI/2} 0" />
       <geometry>
         <box size="${shoulder_pitch_len} ${shoulder_pitch_width} ${shoulder_pitch_height}" />
@@ -89,5 +95,5 @@
     <parent link="shoulder_pitch_link" />
     <child link="elbow_pitch_link" />
-    <origin xyz="0 0 0.11" rpy="0 0 ${M_PI/2}" />
+    <origin xyz="0 0 0.14" rpy="0 0 ${M_PI/2}" />
     <axis xyz="1 0 0" />
     <limit effort="300" velocity="1" lower="-1.57" upper="1.57" />
@@ -99,12 +105,28 @@
         <box size="${elbow_pitch_len} ${elbow_pitch_width} ${elbow_pitch_height}" />
       </geometry>
-      <material name="White" />
+      <material name="Grey" />
+    </visual>
+  </link>
+  <joint name="wrist_pitch_joint" type="revolute">
+    <parent link="elbow_pitch_link" />
+    <child link="wrist_pitch_link" />
+    <origin xyz="0 0 0.22" rpy="0 0 0" />
+    <axis xyz="1 0 0" />
+    <limit effort="300" velocity="1" lower="-1.57" upper="1.57" />
+  </joint>
+  <link name="wrist_pitch_link">
+    <visual>
+      <origin xyz="0 0 0.05" rpy="0 ${M_PI/2} 0" />
+      <geometry>
+        <box size="${wrist_pitch_len} ${wrist_pitch_width} ${wrist_pitch_height}" />
+      </geometry>
+      <material name="Blue" />
     </visual>
   </link>
   <joint name="wrist_roll_joint" type="revolute">
-    <parent link="elbow_pitch_link" />
+    <parent link="wrist_pitch_link" />
     <child link="wrist_roll_link"/>
-    <origin xyz="0 0 0.22" rpy="-${M_PI/2} ${M_PI/2} 0" />
-    <axis xyz="-1 0 0" />
+    <origin xyz="0 0 0.10" rpy="-${M_PI/2} ${M_PI/2} 0" />
+    <axis xyz="1 0 0" />
     <limit effort="300" velocity="1" lower="-1.57" upper="1.57" />
   </joint>
@@ -118,3 +140,35 @@
     </visual>
   </link>
+  <joint name="gripper_left_finger_joint" type="prismatic">
+    <parent link="wrist_roll_link" />
+    <child link="gripper_left_finger_link" />
+    <origin xyz="0 0 0" />
+    <axis xyz="0 1 0" />
+    <limit effort="100" velocity="1" lower="0" upper="0.03" />
+  </joint>
+  <link name="gripper_left_finger_link">
+    <visual>
+      <origin xyz="-0.04 -0.03 0" />
+      <geometry>
+        <box size="${gripper_finger_len} ${gripper_finger_width} ${gripper_finger_height}" />
+      </geometry>
+      <material name="Blue" />
+    </visual>
+  </link>
+  <joint name="gripper_right_finger_joint" type="fixed">
+    <parent link="wrist_roll_link" />
+    <child link="gripper_right_finger_link" />
+    <origin xyz="0 0 0" />
+    <axis xyz="0 1 0" />
+    <!--<limit effort="1" velocity="1" lower="-0.03" upper="0" />-->
+  </joint>
+  <link name="gripper_right_finger_link">
+    <visual>
+      <origin xyz="-0.04 0.03 0" />
+      <geometry>
+        <box size="${gripper_finger_len} ${gripper_finger_width} ${gripper_finger_height}" />
+      </geometry>
+      <material name="Blue" />
+    </visual>
+  </link>
 </robot>
